File: as5045-breakout/as5045-breakout.kicad_pcb (KiCad board)
At the start: 2 copper layers, 17.5 x 72.5 mm, 8 parts, among them P1 CONN_6X2, U1 JMP_3, U2 AS5045

Commit message: work on AS5045 breakout
Parts:
- added ACRO_MOTOR_MOUNT: VAL**, owncomp:ACRO_MOTOR_MOUNT, F.Cu at (60.0, 60.0)
- added C3: 10µ, Capacitors_Tantalum_SMD:TantalC_SizeA_EIA-3216_HandSoldering, F.Cu at (93.5, 73.5)
- added D2: LED (yellow), LEDs:LED-0603, F.Cu at (123.5, 73.4)
- added D3: LED (red), LEDs:LED-0603, F.Cu at (121.3, 73.4)
- added R3: 0, Resistors_SMD:Resistor_SMD1206_HandSoldering, F.Cu at (131.0, 66.0)
- added R4: 680, Resistors_SMD:Resistor_SMD0805_HandSoldering, F.Cu at (123.0, 77.0)
- added U3: LM1117, SMD_Packages:SOT223, F.Cu at (95.0, 65.0)
- C2: footprint SMD_Packages:SM0603_Capa -> Capacitors_Tantalum_SMD:TantalC_SizeA_EIA-3216_HandSoldering
- D1: value LED_BI_COLOR -> LED (green); footprint owncomp:LED_BI_COLOR -> LEDs:LED-0603
- P1: value CONN_6X2 -> CONN_6; footprint owncomp:CONN_6x2 -> owncomp:FLATCONN_6
- R1, R2: footprint SMD_Packages:SM0603_Resistor -> Resistors_SMD:Resistor_SMD0805_HandSoldering
- moved P1 64.9 mm to (95.6, 82.5), turned to 90 degrees
- moved C2 58.8 mm to (96.5, 73.5), turned to 90 degrees
- moved D1 33.6 mm to (125.7, 73.4)
- moved U1 28.3 mm to (128.0, 71.0), turned to 90 degrees
- moved R1 26.5 mm to (129.0, 75.5), turned to 0 degrees
- moved R2 26.2 mm to (129.0, 78.0), turned to 180 degrees
- moved U2 18.1 mm to (135.9, 72.5)
- moved C1 18.1 mm to (131.7, 68.7), turned to 180 degrees
Connections:
- P1 pad 1: VCC -> GND
- P1 pad 2: VCC -> V_IN
- P1 pad 3: GND -> PROG
- P1 pad 4: GND -> DO
- P1 pad 5: PROG -> CLK
- P1 pad 6: PROG -> CSn
- R1 pad 1: Net-(D1-Pad2) -> Net-(D2-Pad2)
- R2 pad 2: Net-(D1-Pad4) -> Net-(D3-Pad2)
Routing:
- net (no net): track 180.0 -> 0.00 mm
- net Net-(R1-Pad2): track 29.6 -> 3.61 mm
- net Net-(R2-Pad1): track 28.7 -> 5.50 mm
- net V_IN: track 0.00 -> 19.7 mm
- net Net-(D3-Pad2): track 0.00 -> 10.2 mm
- net Net-(D1-Pad2): track 2.41 -> 10.3 mm
- net Net-(U1-Pad2): track 5.93 -> 12.3 mm
- net Net-(D2-Pad2): track 0.00 -> 5.37 mm
- net GND: track 60.6 -> 65.5 mm
- net DO: track 67.0 -> 64.5 mm
- net CSn: track 71.5 -> 69.0 mm
- net Net-(D1-Pad4): track 2.41 -> 0.00 mm
- added copper zone on F.Cu, net Net-(U3-Pad4)
Other:
- board outline removed
- net class POWER added: clearance 0.1, trace_width 0.5, via_dia 0.889, via_drill 0.635
- board text added: "www.xrpbot.org"
